File: PSEEL84-chokeload/PSEEL84-chokeload.kicad_sch (KiCad schematic)
At the start: 9 parts, among them U1 ECC88

Commit message: princip scheman
Parts:
- added C3, C4: C_Polarized, symbol Device:C_Polarized
- added C7: C, symbol Device:C
- added D1, D2: D_Zener, symbol Device:D_Zener
- added Q1: DN2540N5-G, Package_TO_SOT_THT:TO-220-3_Vertical, symbol Transistor_FET_Other:DN2540N5-G
- added R1, R2, R3, Rgrid, Rk1, Rk2, Rstop (x2): R, symbol Device:R
- added U2: ECC88, Valve:Valve_Noval_P, symbol Valve:ECC88
Connections:
- net B+: now also U2.1 (A)
- net Earth: now also R2.2, R3.2, Rgrid.2, Rk1.2, Rk2.2
- new net: Rgrid.1, Rstop.1, U2.2 (G)
- new net: C3.1, C4.1, D2.1 (K), Q1.3 (S), R3.1
- new net: D1.2 (A), D2.2 (A)
- new net: C3.2, C4.2
- new net: Q1.1 (G), Rstop.1
- new net: D1.1 (K), R1.2, R2.1, Rstop.2
- new net: C7.2, Rk1.1, U2.3 (K)
- new net: C7.1, Rk2.1
- new net VSS: Q1.2 (D), R1.1
Other:
- note added: "GATE"
- note added: "GATE RAW"
- note added: "IN"
- note added: "In"
- note added: "OUT"
- note added: "OUT NODE"
- note added: "RET"
- note added: "VSS"
