File: PSEEL84-chokeload/PSEEL84-chokeload.kicad_sch (KiCad schematic)
At the start: 24 parts, among them Q1 DN2540N5-G, U1 ECC88, U2 ECC88

Commit message: Lägg till hela my_kicad_work
Parts:
- removed Rstop: R, symbol Device:R
- added Rstop1: R, symbol Device:R
Connections:
- net at U2.2 (G): now also Rstop1.1; no longer Rgrid.1
- net Earth renamed Zero return
- net Zero return: no longer Rgrid.2, Rk1.2, Rk2.2
- new net: Rgrid.1, Rstop1.2
- new net zero: Rgrid.2, Rk1.2, Rk2.2
Other:
- note added: "node ut"
- moved on the sheet: Rgrid
Changed lines of the file:
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@@
+		)
+	)
+	(text "node ut"
+		(exclude_from_sim no)
+		(at 58.928 55.372 0)
+		(effects
+			(font
+				(size 1.27 1.27)
+			)
 		)
 	)
@@
 	)
 	(junction
-		(at 241.3 80.01)
+		(at 231.14 80.01)
 		(diameter 0)
 		(color 0 0 0 0)
@@
 	)
 	(junction
-		(at 241.3 46.99)
+		(at 231.14 46.99)
 		(diameter 0)
 		(color 0 0 0 0)
@@
 	(wire
 		(pts
-			(xy 241.3 46.99) (xy 245.11 46.99)
+			(xy 243.84 46.99) (xy 245.11 46.99)
 		)
 		(stroke
@@
 	(wire
 		(pts
+			(xy 231.14 46.99) (xy 236.22 46.99)
+		)
+		(stroke
+			(width 0)
+			(type default)
+		)
+	)
+	(wire
+		(pts
 			(xy 54.61 45.72) (xy 54.61 27.94)
 		)
@@
 	(wire
 		(pts
-			(xy 240.03 46.99) (xy 241.3 46.99)
-		)
-		(stroke
-			(width 0)
-			(type default)
-		)
-	)
-	(wire
-		(pts
 			(xy 64.77 101.6) (xy 69.85 101.6)
 		)
@@
 	(wire
 		(pts
-			(xy 241.3 80.01) (xy 250.19 80.01)
+			(xy 231.14 80.01) (xy 250.19 80.01)
 		)
 		(stroke
@@
 	(wire
 		(pts
-			(xy 241.3 68.58) (xy 241.3 80.01)
+			(xy 231.14 68.58) (xy 231.14 80.01)
 		)
 		(stroke
@@
 	(wire
 		(pts
-			(xy 241.3 60.96) (xy 241.3 46.99)
+			(xy 231.14 60.96) (xy 231.14 46.99)
 		)
 		(stroke
@@
 	(wire
 		(pts
-			(xy 217.17 80.01) (xy 241.3 80.01)
+			(xy 217.17 80.01) (xy 231.14 80.01)
 		)
 		(stroke
@@
 	(wire
 		(pts
-			(xy 227.33 46.99) (xy 232.41 46.99)
+			(xy 227.33 46.99) (xy 231.14 46.99)
 		)
 		(stroke
@@
 			(width 0)
 			(type default)
-		)
-	)
-	(symbol
-		(lib_id "Device:R")
-		(at 236.22 46.99 270)
-		(unit 1)
-		(exclude_from_sim no)
-		(in_bom yes)
-		(on_board yes)
-		(dnp no)
-		(fields_autoplaced yes)
-		(property "Reference" "Rstop"
-			(at 236.22 40.64 90)
-			(effects
-				(font
-					(size 1.27 1.27)
-				)
-			)
-		)
-		(property "Value" "R"
-			(at 236.22 43.18 90)
-			(effects
-				(font
-					(size 1.27 1.27)
-				)
-			)
-		)
-		(property "Footprint" ""
-			(at 236.22 45.212 90)
-			(effects
-				(font
-					(size 1.27 1.27)
-				)
-				(hide yes)
-			)
-		)
-		(property "Datasheet" "~"
-			(at 236.22 46.99 0)
-			(effects
-				(font
-					(size 1.27 1.27)
-				)
-				(hide yes)
-			)
-		)
-		(property "Description" "Resistor"
-			(at 236.22 46.99 0)
-			(effects
-				(font
-					(size 1.27 1.27)
-				)
-				(hide yes)
-			)
-		)
-		(pin "1"
-		)
-		(pin "2"
-		)
-		(instances
-			(project "PSEEL84-chokeload"
-				(path "/32ca6d0c-12de-40f2-b65a-e4298ae46a02"
-					(reference "Rstop")
-					(unit 1)
-				)
-			)
 		)
 	)
@@
 			)
 		)
-		(property "Value" "Earth"
+		(property "Value" "zero"
 			(at 262.89 85.09 0)
 			(effects
@@
 	(symbol
 		(lib_id "Device:R")
+		(at 240.03 46.99 270)
+		(unit 1)
+		(exclude_from_sim no)
+		(in_bom yes)
+		(on_board yes)
+		(dnp no)
+		(fields_autoplaced yes)
+		(property "Reference" "Rstop1"
+			(at 240.03 40.64 90)
+			(effects
+				(font
+					(size 1.27 1.27)
+				)
+			)
+		)
+		(property "Value" "R"
+			(at 240.03 43.18 90)
+			(effects
+				(font
+					(size 1.27 1.27)
+				)
+			)
+		)
+		(property "Footprint" ""
+			(at 240.03 45.212 90)
+			(effects
+				(font
+					(size 1.27 1.27)
+				)
+				(hide yes)
+			)
+		)
+		(property "Datasheet" "~"
+			(at 240.03 46.99 0)
+			(effects
+				(font
+					(size 1.27 1.27)
+				)
+				(hide yes)
+			)
+		)
+		(property "Description" "Resistor"
+			(at 240.03 46.99 0)
+			(effects
+				(font
+					(size 1.27 1.27)
+				)
+				(hide yes)
+			)
+		)
+		(pin "1"
+		)
+		(pin "2"
+		)
+		(instances
+			(project "PSEEL84-chokeload"
+				(path "/32ca6d0c-12de-40f2-b65a-e4298ae46a02"
+					(reference "Rstop1")
+					(unit 1)
+				)
+			)
+		)
+	)
+	(symbol
+		(lib_id "Device:R")
 		(at 166.37 83.82 0)
 		(unit 1)
@@
 		(on_board yes)
 		(dnp no)
-		(fields_autoplaced yes)
 		(property "Reference" "U2"
 			(at 259.08 45.7199 0)
@@
 		)
 		(property "Value" "ECC88"
-			(at 259.08 48.2599 0)
+			(at 259.588 44.196 0)
 			(effects
 				(font
@@
 				)
 				(justify left)
-				(hide yes)
 			)
 		)
@@
 	(symbol
 		(lib_id "Device:R")
-		(at 241.3 64.77 0)
+		(at 231.14 64.77 0)
 		(unit 1)
 		(exclude_from_sim no)
@@
 		(fields_autoplaced yes)
 		(property "Reference" "Rgrid"
-			(at 243.84 63.4999 0)
+			(at 233.68 63.4999 0)
 			(effects
 				(font
@@
 		)
 		(property "Value" "R"
-			(at 243.84 66.0399 0)
+			(at 233.68 66.0399 0)
 			(effects
 				(font
@@
 		)
 		(property "Footprint" ""
-			(at 239.522 64.77 90)
+			(at 229.362 64.77 90)
 			(effects
 				(font
@@
 		)
 		(property "Datasheet" "~"
-			(at 241.3 64.77 0)
+			(at 231.14 64.77 0)
 			(effects
 				(font
@@
 		)
 		(property "Description" "Resistor"
-			(at 241.3 64.77 0)
+			(at 231.14 64.77 0)
 			(effects
 				(font
@@
 		(on_board yes)
 		(dnp no)
-		(fields_autoplaced yes)
 		(property "Reference" "#PWR02"
 			(at 64.77 107.95 0)
@@
 			)
 		)
-		(property "Value" "Earth"
-			(at 64.77 106.68 0)
-			(effects
-				(font
-					(size 1.27 1.27)
-				)
-			)
-		)
+		(property "Value" "Zero return"
+			(at 61.722 106.172 0)
+			(effects
+				(font
+					(size 1.27 1.27)
+				)
+				(justify left)
+			)
+		)
