File: e-choke/e-choke.kicad_sch (KiCad schematic)
At the start: 9 parts, among them U1 ECC88

Commit message: princip scheman
Parts:
- removed C1, C2: C, symbol Device:C
- removed Ck: ~, symbol Device:C_Polarized
- removed Ck: Ck, symbol Device:C
- removed L1: 200 H, symbol Device:L_Iron
- removed Rgrid, Rk, Rstop: R, symbol Device:R
- removed U1: ECC88, Valve:Valve_Noval_P, symbol Valve:ECC88
- added C2, Cgate: C_Polarized, symbol Device:C_Polarized
- added C3, C4, C5href: C, symbol Device:C
- added D2: D_Zener, symbol Device:D_Zener
- added Q1: 2SK2996, symbol Transistor_FET:Q_NMOS_SGD
- added R5, Rbleeder, Rcharge, Rgatestop: R, symbol Device:R
Connections:
- net Earth: now also C2.2, C3.2, C4.1, C4.2, C5href.1, C5href.2, Cgate.2, Rbleeder.2
- new net: Q1.1 (S), Rbleeder.1
- new net: C2.1, D2.2 (A), Q1.3 (D), R5.1, Rcharge.1
- new net: C3.1, Cgate.1, Rcharge.2, Rgatestop.2
- new net: D2.1 (K), Q1.2 (G), Rgatestop.1
Other:
- note added: "BPLUS_RAW"
- note added: "GATE_REF"
- note added: "VA_BPLUS (VSS_VA)"
