File: gridvoltage_vario/gridvoltage_vario.kicad_sch (KiCad schematic)
At the start: 11 parts, among them U1 MCP4725xxx-xCH, U2 ICL7660, U3 TL072

Commit message: Update gridvoltage_vario schematic
Parts:
- removed R1, R2: 10k, Resistor_THT:R_Axial_DIN0617_L17.0mm_D6.0mm_P25.40mm_Horizontal, symbol Device:R_Small
Connections:
- net Earth: now also U3.3 (+)
- net at U3.5 (+): now also R4.1, U3.1
- net at U3.6 (-), U3.7: no longer U3.3 (+)
