File: ECC83-EL84/ECC83-EL84.kicad_sch (KiCad schematic)
At the start: 14 parts, among them T1 Transformer_1P_1S, U1 ECC83, U2 EL84

Commit message: Lägg till hela my_kicad_work
Other:
- note added: "300 V"
Changed lines of the file:
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@@
 	(generator_version "9.0")
 	(paper "A4")
+	(text "300 V"
+		(exclude_from_sim no)
+		(at 83.058 25.908 0)
+		(effects
+			(font
+				(size 1.27 1.27)
+			)
+		)
+	)
 	(junction
 		(at 186.69 120.65)
