File: Styra_inspänning/Styra_inspänning'.kicad_sch (KiCad schematic)
At the start: 11 parts, among them U1 OPA2134

Commit message: Lägg till hela my_kicad_work
Parts:
- added C5, C6: 10 uF, Capacitor_THT:CP_Radial_D13.0mm_P7.50mm, symbol Device:C_Polarized
- added P1: USB_C_Plug_USB2.0, Connector_USB:USB_C_Receptacle_Amphenol_124019772112A, symbol Connector:USB_C_Plug_USB2.0
- added R5: 5.1 k, Resistor_THT:R_Axial_DIN0614_L14.3mm_D5.7mm_P15.24mm_Horizontal, symbol Device:R
- added U2: ICL7660, Package_DIP:DIP-8_W10.16mm, symbol Regulator_SwitchedCapacitor:ICL7660
- C1, C2, C3, C4: footprint (none) -> Capacitor_THT:CP_Radial_D13.0mm_P7.50mm
- R1, R2, R3, R4: footprint (none) -> Resistor_THT:R_Axial_DIN0614_L14.3mm_D5.7mm_P15.24mm_Horizontal
- RV1: footprint (none) -> Potentiometer_THT:Potentiometer_Bourns_3266Z_Horizontal
- Rsafe1: renamed from Rsafe; footprint (none) -> Resistor_THT:R_Axial_DIN0614_L14.3mm_D5.7mm_P15.24mm_Horizontal
- U1: footprint (none) -> Package_DIP:DIP-8_W10.16mm
Connections:
- net at C1.1, C1.2, C4.2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: now also C6.2, U2.5 (VOUT)
- net at C2.1, C2.2, C3.1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: now also P1.A4 (VBUS), P1.A9 (VBUS), P1.B4 (VBUS), P1.B9 (VBUS), U2.8 (V+)
- net at C3.2, C4.1, R2.2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: now also C6.1, P1.A1 (GND), P1.A12 (GND), P1.B1 (GND), P1.B12 (GND), R5.2, U2.3 (GND)
- new net: C5.1, U2.2 (CAP+)
- new net: C5.2, U2.4 (CAP-)
- new net: P1.A5 (CC), R5.1
Other:
- moved on the sheet: R1, R2, R3, R4
