File: op-amb-labb-2/op-amb-labb-2.kicad_sch (KiCad schematic)
At the start: 7 parts, among them U1 LM358

Commit message: Lägg till hela my_kicad_work
Parts:
- added TP1, TP2, TP3, TP4, TP5: TestPoint, TestPoint:TestPoint_Bridge_Pitch5.08mm_Drill0.7mm, symbol Connector:TestPoint
- C1: footprint (none) -> Capacitor_THT:CP_Axial_L29.0mm_D10.0mm_P35.00mm_Horizontal
- MES1, MES2: footprint (none) -> TestPoint:TestPoint_Bridge_Pitch5.08mm_Drill0.7mm
- RV1: footprint (none) -> Potentiometer_THT:Potentiometer_Vishay_148-149_Single_Vertical
- Rf1: renamed from Rf; value R -> 10 kohm; footprint (none) -> Resistor_THT:R_Axial_DIN0614_L14.3mm_D5.7mm_P15.24mm_Horizontal
- Rg1: renamed from Rg; value R -> 10 kohm; footprint (none) -> Resistor_THT:R_Axial_DIN0614_L14.3mm_D5.7mm_P15.24mm_Horizontal
- U1: footprint (none) -> Package_DIP:CERDIP-8_W7.62mm_SideBrazed
Connections:
- net at MES1.2 (+), Rf1.1, U1.1: now also TP2.1
- net at C1.1, RV1.1, U1.8 (V+): now also TP1.1, TP3.1
- net at C1.2, MES1.1 (-), MES2.1 (-)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: now also TP4.1, TP5.1
