File: 001-elektronik_scheman_labb/opamps_3.0/SHUNT-1.0/SHUNT-1.0.kicad_sch (KiCad schematic)
At the start: 7 parts, among them U1 OPA2277, U2 OPA2277

Commit message: Läge före Konnect
Parts:
- removed R3: R, symbol Device:R
- removed U2: OPA2277, symbol Amplifier_Operational:OPA2277
- added C1: C, symbol Device:C
- added OLED-1: Conn_01x04, symbol Connector_Generic:Conn_01x04
- added R-shunt-2: 1R, symbol Device:R
- added R1, R12, R13, R5, R6: 10K, symbol Device:R
- added R10, R7, R9: 200K, symbol Device:R
- added R8: 200k, symbol Device:R
- added U2: ADS1115IDGS, Package_SO:TSSOP-10_3x3mm_P0.5mm, symbol Analog_ADC:ADS1115IDGS
- R-shunt-1: renamed from R1; value R -> 1R
- R2, R4: value R -> 10K
Connections:
- net at A1.23 (SDA/A4): now also OLED-1.2 (SDA), U2.9 (SDA)
- net at A1.24 (SCL/A5): now also OLED-1.1 (SCL), U2.10 (SCL)
- net at A1.27 (+5V): now also OLED-1.3 (vcc), U2.8 (VDD)
- net GND: now reaches A1.29 (GND), A1.4 (GND)
- net GND: now also R-shunt-1.2, R2.1, C1.2, OLED-1.4 (gnd), R8.1, U2.3 (GND)
- net at R2.2: now also U1.2 (-), R7.2
- net at U1.1: now also R13.2, R7.1
- net at U1.3 (+): now also R1.1, R8.2
- net at R-shunt-1.1: now also R1.2
- new net: C1.1, R13.1, U2.4 (AIN0)
Other:
- moved on the sheet: A1, R-shunt-1, U1A, U1B, U1C
