File: 001-elektronik_scheman_labb/opamps_3.0/op-amp-test-02/_restore_backup_2026-08-31T18-19-04-516/op-amp-test-02.kicad_pcb (KiCad board)
At the start: 2 copper layers, 100 x 55 mm, 24 parts, among them J1 audio-input, J2 audio-output, J3 power_inp, SW1 SW_Rotary_1x5_MP, U2 OPA134

Commit message: Läge före Konnect
Parts:
- removed R1: 100k, Resistor_THT:R_Axial_DIN0207_L6.3mm_D2.5mm_P7.62mm_Horizontal
- added D1: 1N4148, Diode_THT:D_DO-35_SOD27_P7.62mm_Horizontal, F.Cu at (173.0, 66.2)
- added D2: 1N4148, Diode_THT:D_DO-35_SOD27_P7.62mm_Horizontal, F.Cu at (166.0, 73.8)
- added R10: 1k, Resistor_THT:R_Axial_DIN0207_L6.3mm_D2.5mm_P7.62mm_Horizontal, F.Cu at (171.7, 85.0)
- added R9: 10k, Resistor_THT:R_Axial_DIN0207_L6.3mm_D2.5mm_P7.62mm_Horizontal, F.Cu at (199.0, 70.2)
- C6: value 100 pF -> 47 pF
- R8: value 10k -> 100k
Connections:
- C5 pad 1: /OPAMP_IN_P -> /OPAMP_IN
- C6 pad 1: /OPAMP_IN_P -> /OPAMP_IN_3
- R8 pad 1: /OPAMP_IN_P -> /OPAMP_IN_3
- U2 pad 3: /OPAMP_IN_P -> /OPAMP_IN_3
Routing:
- net /OPAMP_IN_P: track 43.7 -> 0.00 mm
- net /OPAMP_IN_3: track 0.00 -> 27.6 mm
- net /OPAMP_IN: track 0.00 -> 20.0 mm
- net /OPAMP_IN_N: track 53.4 -> 62.5 mm
- net /12V-: track 132.5 -> 137.4 mm
- net /12 V+: track 123.4 -> 127.7 mm
