File: 001-elektronik_scheman_labb/opamps_3.0/Dempbox_4.0_relays/relay_1.0_sch.kicad_sch (KiCad schematic)
At the start: 46 parts, among them J5 OLCD_screen, J7 Power, K1 G6K-2, K2 G6K-2, K3 G6K-2, K4 G6K-2, K5 G6K-2, Q1 2N7000, Q2 2N7000, Q3 2N7000, Q4 2N7000, Q5 2N7000, SW2 RotaryEncoder_Switch

Commit message: Backup 2026-10-12
Parts:
- removed J7: Power, symbol Connector:Screw_Terminal_01x02
- added JP1: GND_LINK, Connector_PinHeader_2.54mm:PinHeader_1x02_P2.54mm_Vertical, symbol Jumper:Jumper_2_Open
- A1: value Arduino_Nano_v3.x -> Arduino_Nano_esp32
- C10, C11, C12, C8, C9: footprint Package_SO:SOIC-8_3.9x4.9mm_P1.27mm -> Capacitor_THT:C_Disc_D3.4mm_W2.1mm_P2.50mm
- C13: footprint Package_SO:SOIC-8_3.9x4.9mm_P1.27mm -> Capacitor_THT:C_Disc_D5.0mm_W2.5mm_P5.00mm
- C14: footprint (none) -> Capacitor_THT:CP_Radial_D6.3mm_P2.50mm
- D11, D12, D13, D14, D6: footprint LED_SMD:LED_Cree-XHP50_3V_HighDensity -> LED_THT:LED_D3.0mm
- J5: footprint Package_SON:WSON-8-1EP_6x5mm_P1.27mm_EP3.4x4mm -> Connector_PinSocket_2.54mm:PinSocket_1x04_P2.54mm_Vertical
- K1, K2, K3, K4, K5: footprint Relay_THT:Relay_StandexMeder_DIP_LowProfile -> Relay_THT:Relay_DPDT_Omron_G6K-2P; symbol Relay:DIPxx-1Axx-13x -> Relay:G6K-2
- R1, R11, R2, R27, R28, R29, R3, R30, R31, R32, R33, R4, R5, R6, R8: footprint (none) -> Resistor_THT:R_Axial_DIN0204_L3.6mm_D1.6mm_P7.62mm_Horizontal
- SW2: footprint (none) -> Rotary_Encoder:RotaryEncoder_Alps_EC11E-Switch_Vertical_H20mm
Connections:
- net GND is gone; now on net power ground: C13.2, C14.2, Q1.1 (S), Q2.1 (S), Q3.1 (S), Q4.1 (S), Q5.1 (S), R11.1, R2.1, R28.1, R4.1, R6.1
- net INT_1_100_OUT: now also K1.4; no longer K1.8
- net INT_1_10_OUT: now also K2.4; no longer K2.8
- net LOW_1_1_OUT: now also K5.4; no longer K5.8
- net MEASURE_SIGNAL: now also K1.3, K2.3, K3.3, K4.3, K5.3; no longer K1.14, K2.14, K3.14, K4.14, K5.14
- net Power 5v: now also A1.27 (+5V), J5.4 (Pin_4), K1.1, K2.1, K3.1, K4.1, K5.1; no longer K1.6, K2.6, K3.6, K4.6, K5.6
- net SPK_1_100_OUT: now also K3.4; no longer K3.8
- net SPK_1_10_OUT: now also K4.4; no longer K4.8
- net at C10.2, D3.2 (A), Q3.3 (D)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: now also K3.8; no longer K3.2
- net at C8.2, D5.2 (A), Q5.3 (D)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: now also K5.8; no longer K5.2
- net at C11.2, D2.2 (A), Q2.3 (D)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: now also K2.8; no longer K2.2
- net at C12.2, D1.2 (A), Q1.3 (D)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: now also K1.8; no longer K1.2
- net at C9.2, D4.2 (A), Q4.3 (D)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: now also K4.8; no longer K4.2
- net at A1.15 (D12), R3.2: no longer R1.2
- net power ground: now reaches A1.29 (GND), J5.3 (Pin_3), SW2.S2
- net power ground: now also A1.4 (GND), SW2.C, JP1.1 (A)
- net at A1.23 (A4): now also J5.1 (Pin_1); no longer J5.SCL (Pin_2)
- net at A1.24 (A5): now also J5.2 (Pin_2); no longer J5.SDA (Pin_1)
- net at A1.16 (D13): now also R1.2
- new net MEASURE_GND: JP1.2 (B)
- no-connect marks 18 -> 37
Other:
- moved on the sheet: R1
