File: 001-elektronik_scheman_labb/opamps_3.0/dempbox_relay_7.0/dempbox_relay_7.0.kicad_pcb (KiCad board)
At the start: 2 copper layers, 100 x 100 mm, 86 parts, among them J1 Test_probe, J10 Mätinstrument, J2 TO_Focusrite_input, J3 OP_AMP_PWR, J4 Speaker, J5 OLCD_screen, J9 Mätinstrument, K1 HE721A0500, K2 HE721A0500, K3 HE721A0500, K4 HE721A0500, K5 HE721A0500, Q1 2N7000, Q2 2N7000, Q3 2N7000, Q4 2N7000, Q5 2N7000, SW2 RotaryEncoder_Switch, U2 OPA134

Commit message: Backup 2026-10-18
Parts:
- moved C4 28.0 mm to (153.7, 101.5), turned to -90 degrees
- moved C3 8.35 mm to (165.3, 112.0)
Routing:
- net /sound-card/12V-: track 0.00 -> 70.3 mm, vias 0 -> 1
- net /sound-card/12V+: track 0.00 -> 53.9 mm, vias 0 -> 3
- net SPK_1_10_OUT: track 0.00 -> 40.7 mm, vias 0 -> 2
- net /sound-card/audio_out: track 0.00 -> 37.0 mm
- net LOW_1_1_OUT: track 86.7 -> 57.9 mm, vias 3 -> 4
- net /sound-card/OP_AMP_OUT: track 8.67 -> 18.0 mm
