File: 001-elektronik_scheman_labb/opamps_3.0/volum_control_arduino-1.0/volum_control_arduino-1.0.kicad_pcb (KiCad board)
At the start: 4 copper layers, 100 x 87 mm, 66 parts, among them J1 POWER, J2 MAIN_IN, J3 SUB_IN, J4 MAIN_OUT, J5 SUB_OUT, J6 ISP, SW1 EC11, U1 PGA2311PA, U2 PGA2311PA, U3 OPA2134PA, U4 OPA2134PA, U5 ATmega328P-P, U6 TSOP38238, U7 L7805, U8 L7905, Y1 16MHz

Commit message: Backup 2026-10-18
Parts:
- removed C28, C29, C30, C33: 100nF, Capacitor_THT:C_Disc_D5.0mm_W2.5mm_P2.50mm
- removed C31, C32: 22pF, Capacitor_THT:C_Disc_D5.0mm_W2.5mm_P2.50mm
- removed J6: ISP, Connector_PinHeader_2.54mm:PinHeader_2x03_P2.54mm_Vertical
- removed R10: 10k, Resistor_THT:R_Axial_DIN0207_L6.3mm_D2.5mm_P7.62mm_Horizontal
- removed U5: ATmega328P-P, Package_DIP:DIP-28_W7.62mm
- removed Y1: 16MHz, Crystal:Crystal_HC49-U_Vertical
- added A1: Arduino_Nano, Module:Arduino_Nano, F.Cu at (142.2, 134.0)
- added C35: 10uF, Capacitor_THT:CP_Radial_D5.0mm_P2.00mm, F.Cu at (149.0, 64.0)
- added C36: 10uF, Capacitor_THT:CP_Radial_D5.0mm_P2.00mm, F.Cu at (155.0, 64.0)
- added C37: 100nF, Capacitor_THT:C_Disc_D5.0mm_W2.5mm_P2.50mm, F.Cu at (158.5, 64.0)
- added C38: 100uF, Capacitor_THT:CP_Radial_D6.3mm_P2.50mm, F.Cu at (142.6, 58.0)
- added C39: 100nF, Capacitor_THT:C_Disc_D5.0mm_W2.5mm_P2.50mm, F.Cu at (141.0, 68.5)
- added D2: 1N4148, Diode_THT:D_DO-35_SOD27_P7.62mm_Horizontal, F.Cu at (165.0, 135.5)
- added D3: 1N4148, Diode_THT:D_DO-35_SOD27_P7.62mm_Horizontal, F.Cu at (179.0, 135.5)
- added D4: 1N4148, Diode_THT:D_DO-35_SOD27_P7.62mm_Horizontal, F.Cu at (193.0, 135.5)
- added H1: MountingHole, MountingHole:MountingHole_3.2mm, F.Cu at (196.0, 52.0)
- added H2: MountingHole, MountingHole:MountingHole_3.2mm, F.Cu at (196.0, 148.0)
- added H3: MountingHole, MountingHole:MountingHole_3.2mm, F.Cu at (150.0, 148.0)
- added H4: MountingHole, MountingHole:MountingHole_3.2mm, F.Cu at (103.5, 51.5)
- added J7: RELAYS, Connector_PinHeader_2.54mm:PinHeader_1x04_P2.54mm_Vertical, F.Cu at (172.0, 149.6)
- added Q1: BC547, Package_TO_SOT_THT:TO-92_Inline, F.Cu at (161.5, 141.0)
- added Q2: BC547, Package_TO_SOT_THT:TO-92_Inline, F.Cu at (175.5, 141.0)
- added Q3: BC547, Package_TO_SOT_THT:TO-92_Inline, F.Cu at (189.5, 141.0)
- added R16: 10k, Resistor_THT:R_Axial_DIN0207_L6.3mm_D2.5mm_P7.62mm_Horizontal, F.Cu at (154.1, 70.0)
- added R17: 4.7k, Resistor_THT:R_Axial_DIN0207_L6.3mm_D2.5mm_P7.62mm_Horizontal, F.Cu at (154.0, 143.1)
- added R18: 100k, Resistor_THT:R_Axial_DIN0207_L6.3mm_D2.5mm_P7.62mm_Horizontal, F.Cu at (157.0, 135.5)
- added R19: 4.7k, Resistor_THT:R_Axial_DIN0207_L6.3mm_D2.5mm_P7.62mm_Horizontal, F.Cu at (168.0, 143.1)
- added R20: 100k, Resistor_THT:R_Axial_DIN0207_L6.3mm_D2.5mm_P7.62mm_Horizontal, F.Cu at (171.0, 135.5)
- added R21: 4.7k, Resistor_THT:R_Axial_DIN0207_L6.3mm_D2.5mm_P7.62mm_Horizontal, F.Cu at (182.0, 143.1)
- added R22: 100k, Resistor_THT:R_Axial_DIN0207_L6.3mm_D2.5mm_P7.62mm_Horizontal, F.Cu at (185.0, 135.5)
- added U10: LD1117V33, Package_TO_SOT_THT:TO-220-3_Vertical, F.Cu at (152.0, 57.0)
- added U9: nRF24L01+PA+LNA, RF_Module:nRF24L01_Breakout, F.Cu at (138.0, 64.0)
- moved J1 81.8 mm to (165.0, 66.0), turned to 90 degrees
- moved D1 72.4 mm to (195.5, 81.5), turned to -90 degrees
- moved C1 70.7 mm to (165.0, 74.0)
- moved C2 70.7 mm to (160.5, 74.0)
- moved C3 70.7 mm to (173.0, 74.0)
- moved C4 70.7 mm to (176.5, 74.0)
- moved U7 70.7 mm to (164.0, 81.0)
- moved U4 67.2 mm to (127.0, 128.0), turned to 180 degrees
- moved U2 54.6 mm to (145.0, 128.0), turned to 180 degrees
- moved U1 50.5 mm to (145.0, 94.0), turned to 180 degrees
- moved C5 40.5 mm to (170.5, 90.0)
- moved C6 40.5 mm to (161.0, 90.0)
- moved C7 40.5 mm to (173.5, 90.0)
- moved C8 40.5 mm to (181.5, 90.0)
- moved U8 40.5 mm to (172.0, 97.0)
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Routing:
- net +12V: track 0.00 -> 233.6 mm, vias 0 -> 15
- net +5V: track 0.00 -> 187.5 mm, vias 0 -> 12
- net +5VA: track 0.00 -> 138.6 mm, vias 0 -> 8
- net -12V: track 0.00 -> 131.7 mm, vias 0 -> 7
- net /SCK: track 0.00 -> 124.0 mm, vias 0 -> 6
- net -5VA: track 0.00 -> 121.8 mm, vias 0 -> 7
- net /NRF_IRQ: track 0.00 -> 103.3 mm, vias 0 -> 2
- net /MISO: track 0.00 -> 98.1 mm
- net /MOSI: track 0.00 -> 94.5 mm, vias 0 -> 2
- net /IR_OUT: track 0.00 -> 93.2 mm, vias 0 -> 1
- net /LED_MUTE: track 0.00 -> 91.7 mm, vias 0 -> 2
- net /NRF_CSN: track 0.00 -> 88.6 mm, vias 0 -> 3
- net /NRF_CE: track 0.00 -> 79.3 mm, vias 0 -> 3
- net /MUTE: track 0.00 -> 78.5 mm, vias 0 -> 5
- net /ENC_SW: track 0.00 -> 78.1 mm
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- added copper zone on In1.Cu, net GND
- added copper zone on In2.Cu, net GND
Other:
- board size 100 x 87 mm -> 100 x 104 mm
