File: 001-elektronik_scheman_labb/opamps_3.0/volum_control_arduino-1.0/volum_control_arduino-1.0.kicad_sch (KiCad schematic)
At the start: 66 parts, among them J1 POWER, J2 MAIN_IN, J3 SUB_IN, J4 MAIN_OUT, J5 SUB_OUT, J6 ISP, SW1 EC11, U1 PGA2311PA, U2 PGA2311PA, U3 OPA2134PA, U4 OPA2134PA, U5 ATmega328P-P, U6 TSOP38238, U7 L7805, U8 L7905, Y1 16MHz

Commit message: Backup 2026-10-18
Parts:
- removed C28, C29, C30, C33: 100nF, Capacitor_THT:C_Disc_D5.0mm_W2.5mm_P2.50mm, symbol Device:C
- removed C31, C32: 22pF, Capacitor_THT:C_Disc_D5.0mm_W2.5mm_P2.50mm, symbol Device:C
- removed J6: ISP, Connector_PinHeader_2.54mm:PinHeader_2x03_P2.54mm_Vertical, symbol Connector:AVR-ISP-6
- removed R10: 10k, Resistor_THT:R_Axial_DIN0207_L6.3mm_D2.5mm_P7.62mm_Horizontal, symbol Device:R
- removed U5: ATmega328P-P, Package_DIP:DIP-28_W7.62mm, symbol MCU_Microchip_ATmega:ATmega328P-P
- removed Y1: 16MHz, Crystal:Crystal_HC49-U_Vertical, symbol Device:Crystal
- added A1: Arduino_Nano, Module:Arduino_Nano, symbol MCU_Module:Arduino_Nano_v3.x
- added C35, C36: 10uF, Capacitor_THT:CP_Radial_D5.0mm_P2.00mm, symbol Device:C_Polarized
- added C37, C39: 100nF, Capacitor_THT:C_Disc_D5.0mm_W2.5mm_P2.50mm, symbol Device:C
- added C38: 100uF, Capacitor_THT:CP_Radial_D6.3mm_P2.50mm, symbol Device:C_Polarized
- added D2, D3, D4: 1N4148, Diode_THT:D_DO-35_SOD27_P7.62mm_Horizontal, symbol Diode:1N4148
- added J7: RELAYS, Connector_PinHeader_2.54mm:PinHeader_1x04_P2.54mm_Vertical, symbol Connector_Generic:Conn_01x04
- added Q1, Q2, Q3: BC547, Package_TO_SOT_THT:TO-92_Inline, symbol Transistor_BJT:BC547
- added R16: 10k, Resistor_THT:R_Axial_DIN0207_L6.3mm_D2.5mm_P7.62mm_Horizontal, symbol Device:R
- added R17, R19, R21: 4.7k, Resistor_THT:R_Axial_DIN0207_L6.3mm_D2.5mm_P7.62mm_Horizontal, symbol Device:R
- added R18, R20, R22: 100k, Resistor_THT:R_Axial_DIN0207_L6.3mm_D2.5mm_P7.62mm_Horizontal, symbol Device:R
- added U10: LD1117V33, Package_TO_SOT_THT:TO-220-3_Vertical, symbol Regulator_Linear:LD1117V33
- added U9: nRF24L01+PA+LNA, RF_Module:nRF24L01_Breakout, symbol RF:NRF24L01_Breakout
Connections:
- net +12V: now also C35.1, D2.1 (K), D3.1 (K), D4.1 (K), J7.1 (Pin_1), U10.3 (VI)
- net +5V: now also A1.27 (+5V)
- net ENC_A: now also A1.6 (D3)
- net ENC_B: now also A1.7 (D4)
- net ENC_SW: now also A1.8 (D5)
- net GND: now also A1.29 (GND), A1.4 (GND), C35.2, C36.2, C37.2, C38.2, C39.2, Q1.3 (E), Q2.3 (E), Q3.3 (E), R18.2, R20.2, R22.2, U10.1 (GND), U9.1 (GND)
- net IR_OUT: now also A1.5 (D2)
- net LED_MUTE: now also A1.11 (D8)
- net MISO: now also A1.15 (D12), U9.7 (MISO)
- net MOSI: now also A1.14 (D11), U9.6 (MOSI)
- net MUTE: now also A1.12 (D9)
- net PGA_CS: now also A1.13 (D10)
- net SCK: now also A1.16 (D13), U9.5 (SCK)
- new net: Q1.2 (B), R17.2, R18.1
- new net: Q2.2 (B), R19.2, R20.1
- new net: Q3.2 (B), R21.2, R22.1
- new net +3V3: C36.1, C37.1, C38.1, C39.1, R16.1, U10.2 (VO), U9.2 (VCC)
- new net NRF_CE: A1.10 (D7), U9.3 (CE)
- new net NRF_CSN: A1.9 (D6), R16.2, U9.4 (~{CSN})
- new net NRF_IRQ: A1.19 (A0), U9.8 (IRQ)
- new net RLY1: D2.2 (A), J7.2 (Pin_2), Q1.1 (C)
- new net RLY2: D3.2 (A), J7.3 (Pin_3), Q2.1 (C)
- new net RLY3: D4.2 (A), J7.4 (Pin_4), Q3.1 (C)
- new net RLY_CTRL1: A1.20 (A1), R17.1
- new net RLY_CTRL2: A1.21 (A2), R19.1
- new net RLY_CTRL3: A1.22 (A3), R21.1
- no-connect marks 12 -> 13
